Commit message: Add orca_gz package, refactor

File: orca_bringup/urdf/orca5_1.urdf (robot description, URDF)
Before this commit: robot orca5_1, 3 links, 2 joints
Links:
- link base_link: geometry collision box size=0.457 0.338 0.0673; visual mesh filename=package://orca_bringup/urdf/meshes/bluerov2.dae scale=0.025 0.025 0.025
